File: cr3-power-regulator.kicad_sch (KiCad schematic)
At the start: 11 parts, among them J1 Conn_01x06_Female, U1 L7812, U2 L7912

Commit message: Update footprints
- 1mm headder was accidentally used instead of 2.54mm (.1")
- Regulators have correct footprint
- Capacitors updated to use polarized footprints (in case it matters)
Parts:
- C1, C2, C3, C4: footprint Capacitor_THT:C_Disc_D5.1mm_W3.2mm_P5.00mm -> Capacitor_THT:CP_Radial_Tantal_D5.0mm_P2.50mm
- J1: footprint Connector_PinHeader_1.00mm:PinHeader_1x06_P1.00mm_Horizontal -> Connector_PinHeader_2.54mm:PinHeader_1x06_P2.54mm_Vertical
- U1, U2: footprint Connector_PinHeader_1.00mm:PinHeader_1x03_P1.00mm_Horizontal -> Package_TO_SOT_THT:TO-220-3_Vertical
Changed lines of the file:
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@@
       (effects (font (size 1.27 1.27)) (justify left))
     )
-    (property "Footprint" "Capacitor_THT:C_Disc_D5.1mm_W3.2mm_P5.00mm" (id 2) (at 76.2 80.01 0)
+    (property "Footprint" "Capacitor_THT:CP_Radial_Tantal_D5.0mm_P2.50mm" (id 2) (at 76.2 80.01 0)
       (effects (font (size 1.27 1.27)) hide)
     )
@@
       (effects (font (size 1.27 1.27)) (justify left))
     )
-    (property "Footprint" "Capacitor_THT:C_Disc_D5.1mm_W3.2mm_P5.00mm" (id 2) (at 138.43 78.74 0)
+    (property "Footprint" "Capacitor_THT:CP_Radial_Tantal_D5.0mm_P2.50mm" (id 2) (at 138.43 78.74 0)
       (effects (font (size 1.27 1.27)) hide)
     )
@@
       (effects (font (size 1.27 1.27)) (justify left))
     )
-    (property "Footprint" "Capacitor_THT:C_Disc_D5.1mm_W3.2mm_P5.00mm" (id 2) (at 76.2 67.31 0)
+    (property "Footprint" "Capacitor_THT:CP_Radial_Tantal_D5.0mm_P2.50mm" (id 2) (at 76.2 67.31 0)
       (effects (font (size 1.27 1.27)) hide)
     )
@@
     (property "Reference" "U2" (id 0) (at 101.6 90.17 0))
     (property "Value" "L7912" (id 1) (at 101.6 92.71 0))
-    (property "Footprint" "Connector_PinHeader_1.00mm:PinHeader_1x03_P1.00mm_Horizontal" (id 2) (at 101.6 90.17 0)
+    (property "Footprint" "Package_TO_SOT_THT:TO-220-3_Vertical" (id 2) (at 101.6 90.17 0)
       (effects (font (size 1.27 1.27) italic) hide)
     )
@@
     (property "Reference" "U1" (id 0) (at 101.6 53.34 0))
     (property "Value" "L7812" (id 1) (at 101.6 55.88 0))
-    (property "Footprint" "Connector_PinHeader_1.00mm:PinHeader_1x03_P1.00mm_Horizontal" (id 2) (at 102.235 64.77 0)
+    (property "Footprint" "Package_TO_SOT_THT:TO-220-3_Vertical" (id 2) (at 102.235 64.77 0)
       (effects (font (size 1.27 1.27) italic) (justify left) hide)
     )
@@
       (effects (font (size 1.27 1.27)) (justify left))
     )
-    (property "Footprint" "Capacitor_THT:C_Disc_D5.1mm_W3.2mm_P5.00mm" (id 2) (at 138.43 66.04 0)
+    (property "Footprint" "Capacitor_THT:CP_Radial_Tantal_D5.0mm_P2.50mm" (id 2) (at 138.43 66.04 0)
       (effects (font (size 1.27 1.27)) hide)
     )
@@
       (effects (font (size 1.27 1.27)) (justify left))
     )
-    (property "Footprint" "Connector_PinHeader_1.00mm:PinHeader_1x06_P1.00mm_Horizontal" (id 2) (at 167.64 71.12 0)
+    (property "Footprint" "Connector_PinHeader_2.54mm:PinHeader_1x06_P2.54mm_Vertical" (id 2) (at 167.64 71.12 0)
       (effects (font (size 1.27 1.27)) hide)
     )
@@
     )
     (path "/831bf933-e146-4a93-98fd-133a632bb36e"
-      (reference "C1") (unit 1) (value "100n") (footprint "Capacitor_THT:C_Disc_D5.1mm_W3.2mm_P5.00mm")
+      (reference "C1") (unit 1) (value "100n") (footprint "Capacitor_THT:CP_Radial_Tantal_D5.0mm_P2.50mm")
     )
     (path "/536ee831-5a0f-4a31-80bb-cfd73d7b65ef"
-      (reference "C2") (unit 1) (value "100n") (footprint "Capacitor_THT:C_Disc_D5.1mm_W3.2mm_P5.00mm")
+      (reference "C2") (unit 1) (value "100n") (footprint "Capacitor_THT:CP_Radial_Tantal_D5.0mm_P2.50mm")
     )
     (path "/ca65b035-22c4-4abf-bcef-9ac3ee1485a5"
-      (reference "C3") (unit 1) (value "100n") (footprint "Capacitor_THT:C_Disc_D5.1mm_W3.2mm_P5.00mm")
+      (reference "C3") (unit 1) (value "100n") (footprint "Capacitor_THT:CP_Radial_Tantal_D5.0mm_P2.50mm")
     )
     (path "/57581ba9-98d2-4d29-8a7c-fcb8aaf2cac1"
-      (reference "C4") (unit 1) (value "100n") (footprint "Capacitor_THT:C_Disc_D5.1mm_W3.2mm_P5.00mm")
+      (reference "C4") (unit 1) (value "100n") (footprint "Capacitor_THT:CP_Radial_Tantal_D5.0mm_P2.50mm")
     )
     (path "/57d0436e-f7e8-451c-85bf-f9642b19f779"
@@
     )
     (path "/cb44949c-0065-4af2-a672-d6236f0f00a2"
-      (reference "J1") (unit 1) (value "Conn_01x06_Female") (footprint "Connector_PinHeader_1.00mm:PinHeader_1x06_P1.00mm_Horizontal")
+      (reference "J1") (unit 1) (value "Conn_01x06_Female") (footprint "Connector_PinHeader_2.54mm:PinHeader_1x06_P2.54mm_Vertical")
     )
     (path "/ab570998-d1e0-4e37-86d3-7a6af0c05945"
-      (reference "U1") (unit 1) (value "L7812") (footprint "Connector_PinHeader_1.00mm:PinHeader_1x03_P1.00mm_Horizontal")
+      (reference "U1") (unit 1) (value "L7812") (footprint "Package_TO_SOT_THT:TO-220-3_Vertical")
     )
     (path "/a321fea4-5669-4b00-b6fb-18121dadbb39"
-      (reference "U2") (unit 1) (value "L7912") (footprint "Connector_PinHeader_1.00mm:PinHeader_1x03_P1.00mm_Horizontal")
-    )
-  )
+      (reference "U2") (unit 1) (value "L7912") (footprint "Package_TO_SOT_THT:TO-220-3_Vertical")
+    )
+  )
